Commit message: modify

File: master_robot/urdf/master_robot.urdf (robot description, URDF)
Before this commit: robot my_robot, 8 links, 7 joints
Links:
- added link imu_link; visual box size=0.02 0.047 0.008
Joints:
- added joint imu_link_joint: type fixed, parent base_link, child imu_link, origin xyz=-0.1 -0.06 0.143 rpy=0 0 1.570796
- joint wheel_left_joint: type fixed -> continuous
- joint wheel_right_joint: type fixed -> continuous
